File: Eagle/KVM Keyboard.brd (EAGLE design)
At the start: 460.8 x 147.5 mm, 284 parts

Commit message: Bringing things up to date
Parts:
- moved RGB_BRACE-CLOSING 4.75 mm to (275.5, 66.5)
- moved RGB_BRACE-OPENING 4.75 mm to (256.5, 66.5)
- moved RGB_COLON 4.75 mm to (242.2, 47.5)
- moved RGB_GREATER-THAN 4.75 mm to (232.8, 28.5)
- moved RGB_HOME 4.75 mm to (346.8, 85.5)
- moved RGB_L 4.75 mm to (223.2, 47.5)
- moved RGB_LESS-THAN 4.75 mm to (213.8, 28.5)
- moved RGB_NUM-MINUS 4.75 mm to (247.0, 85.5)
- moved RGB_NUM-PLUS 4.75 mm to (266.0, 85.5)
- moved RGB_NUM0 4.75 mm to (228.0, 85.5)
- moved RGB_NUM9 4.75 mm to (209.0, 85.5)
- moved RGB_O 4.75 mm to (218.5, 66.5)
- moved RGB_P 4.75 mm to (237.5, 66.5)
- moved RGB_QUESTION-MARK 4.75 mm to (251.8, 28.5)
- moved RGB_QUOTATION-MARK 4.75 mm to (261.2, 47.5)
