File: Eagle/Computer Power Relay/Computer Power Relay - Power Strip - Backup.brd (EAGLE design)
At the start: 79.5 x 78 mm, 5 parts, among them K1 RELAY-3V3DC-110VAC012, K3 RELAY-110VACV3_IN-PLACE

Commit message: Beginning Merge of Boards (Relay)
I'm beginning to merge the Controller and Power Strip boards into one so that I can print it for cheaper.
Parts:
- removed U$3: MAINS-POWER-OUTLET3-PIN, Inventory:3-PIN-POWER
- added K2: RELAY-110VACV3_IN-PLACE, Inventory:RELAY-110VAC-V3
- K3: value RELAY-110VACV3_IN-PLACE -> RELAY-110VACV3_SMD; device Inventory:RELAY-110VAC-V3 -> Inventory:RELAY-110VAC-V3-SMD
- U$1: value AUDIO_JACK_FEMALE_5-PIN -> MAINS-POWER-OUTLET3-PIN; device Inventory:AUDIO_JACK_FEMALE_5-PIN -> Inventory:3-PIN-POWER
- moved K1 158.3 mm to (19.1, 209.6), turned to 180 degrees
- moved K3 84.7 mm to (-11.0, -33.6), turned to 0 degrees
- moved U$2 37.1 mm to (2.55, -13.9), turned to 0 degrees
- moved U$1 15.8 mm to (2.55, -6.19), turned to 0 degrees
Connections:
- net RELAY_EN renamed N$14
- removed net 5V: U$1.4, U$1.5
- removed net HOT-SOURCE: K1.1, K3.5, K3.6, U$3.HOT
- removed net N$2: K3.7, U$2.NEUTRAL, U$3.NEUTRAL
- new net N$11: K1.1, K3.5, K3.6, U$2.HOT
- new net N$12: K3.7, U$1.NEUTRAL, U$2.NEUTRAL
- net 3V3_EN: no longer U$1.1, U$1.2
- net GND: now also U$1.GND; no longer U$3.GND
- net GND2: no longer U$1.3
- net N$1: now also U$1.HOT; no longer U$2.HOT
Routing:
- net HOT-SOURCE: track 93.7 -> 0.00 mm
- net GND2: track 83.9 -> 0.00 mm, vias 1 -> 0
- net 3V3_EN: track 54.1 -> 0.00 mm, vias 1 -> 0
- net N$1: track 35.2 -> 0.00 mm
- net 5V: track 24.1 -> 0.00 mm, vias 1 -> 0
- net N$14: track 22.7 -> 0.00 mm
- net N$2: track 10.9 -> 0.00 mm
Other:
- board size 79.5 x 78 mm -> 44.4 x 247.7 mm
- board text removed: "3V3_EN"
- board text removed: "5V"
- board text removed: "GND"
