File: Eagle/Computer Power Relay/Computer Power Relay - Power Strip.brd (EAGLE design)
At the start: 44.4 x 247.7 mm, 6 parts, among them K1 RELAY-3V3DC-110VAC012, K3 RELAY-110VACFLAT-PINS-V2

Commit message: Split controller from power splitter
Parts:
- added U$1: AUDIO_JACK_FEMALE_5-PIN, Inventory:AUDIO_JACK_FEMALE_5-PIN
- moved K3 224.9 mm to (16.8, -53.4), turned to 90 degrees
- moved U$6 58.2 mm to (0.00, 78.4), turned to 270 degrees
- moved U$5 47.0 mm to (0.00, 52.2), turned to 270 degrees
- moved U$4 36.4 mm to (0.00, 26.1), turned to 270 degrees
- moved U$3 26.9 mm to (0.00, 0.00), turned to 270 degrees
- moved K1 25.1 mm to (2.67, 190.5), flipped to the bottom
Connections:
- removed net N$10: K3.3, U$3.NEUTRAL, U$4.NEUTRAL, U$5.NEUTRAL, U$6.NEUTRAL
- removed net N$11: K1.1, K3.2
- removed net N$12: K3.1, K3.7
- removed net N$14: K1.2, K3.8
- removed net N$6: K3.4, U$3.HOT, U$4.HOT, U$5.HOT, U$6.HOT
- new net 5V: U$1.4, U$1.5
- new net HOT: K3.3, K3.4, U$3.NEUTRAL, U$4.NEUTRAL, U$5.NEUTRAL, U$6.NEUTRAL
- new net HOT-RELAY: K1.2, K3.5, K3.6, K3.8
- new net HOT-SOURCE: K1.1
- new net NEUTRAL: K3.7, U$3.HOT, U$4.HOT, U$5.HOT, U$6.HOT
- net 3V3_EN: now also U$1.1, U$1.2
- net GND2: now also U$1.3
Routing:
- net GND2: track 0.00 -> 2083.3 mm, vias 0 -> 1
- net HOT: track 0.00 -> 27.7 mm
- net NEUTRAL: track 0.00 -> 19.9 mm
- net N$38: track 0.00 -> 17.2 mm
- net HOT-RELAY: track 0.00 -> 13.1 mm
- net HOT-SOURCE: track 0.00 -> 13.0 mm
- net 5V: track 0.00 -> 10.0 mm, vias 0 -> 1
- net 3V3_EN: track 0.00 -> 10.0 mm, vias 0 -> 1
- net N$34: track 0.00 -> 6.42 mm
- net N$8: track 0.00 -> 4.39 mm
- net N$33: track 0.00 -> 3.34 mm
- net N$32: track 0.00 -> 3.34 mm
- net N$31: track 0.00 -> 1.05 mm
- net N$23: track 0.00 -> 1.05 mm
- net N$7: track 0.00 -> 0.53 mm
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Other:
- board size 44.4 x 247.7 mm -> 46.4 x 293.7 mm
- board text added: "3V3_EN"
- board text added: "5V"
- board text added: "Common"
- board text added: "GND"
- board text added: "Powered"
- board text added: "Unpowered"

Commit message: Beginning Merge of Boards (Relay)
I'm beginning to merge the Controller and Power Strip boards into one so that I can print it for cheaper.
Parts:
- removed U$4, U$5, U$6: MAINS-POWER-OUTLET, KVM Keyboard:MAINS-POWER-OUTLET
- added U$2: MAINS-POWER-OUTLET3-PIN, Inventory:3-PIN-POWER
- K3: value RELAY-110VACFLAT-PINS-V2 -> RELAY-110VACV3_IN-PLACE; device Inventory:RELAY-110VAC-V2 -> Inventory:RELAY-110VAC-V3
- U$3: value MAINS-POWER-OUTLET -> MAINS-POWER-OUTLET3-PIN; device KVM Keyboard:MAINS-POWER-OUTLET -> Inventory:3-PIN-POWER
- moved K1 142.5 mm to (37.2, 52.3), flipped to the top, turned to 270 degrees
- moved K3 79.5 mm to (59.2, 13.8)
- moved U$3 70.6 mm to (69.2, 13.8)
- moved U$1 63.3 mm to (9.00, 8.28), turned to 270 degrees
Connections:
- removed net HOT: K3.3, K3.4, U$3.NEUTRAL, U$4.NEUTRAL, U$5.NEUTRAL, U$6.NEUTRAL
- removed net HOT-RELAY: K1.2, K3.5, K3.6, K3.8
- removed net N$9: U$3.GND, U$4.GND, U$5.GND, U$6.GND
- removed net NEUTRAL: K3.7, U$3.HOT, U$4.HOT, U$5.HOT, U$6.HOT
- new net GND: U$2.GND, U$3.GND
- new net N$1: K3.3, K3.4, U$2.HOT
- new net N$2: K3.7, U$2.NEUTRAL, U$3.NEUTRAL
- new net RELAY_EN: K1.2, K3.8
- net HOT-SOURCE: now also K3.5, K3.6, U$3.HOT
Routing:
- net GND2: track 2083.3 -> 83.9 mm
- net HOT-SOURCE: track 13.0 -> 93.7 mm
- net 3V3_EN: track 10.0 -> 54.1 mm
- net N$1: track 0.00 -> 35.2 mm
- net HOT: track 27.7 -> 0.00 mm
- net RELAY_EN: track 0.00 -> 22.7 mm
- net NEUTRAL: track 19.9 -> 0.00 mm
- net N$38: track 17.2 -> 0.00 mm
- net 5V: track 10.0 -> 24.1 mm
- net HOT-RELAY: track 13.1 -> 0.00 mm
- net N$2: track 0.00 -> 10.9 mm
- net N$34: track 6.42 -> 0.00 mm
- net N$8: track 4.39 -> 0.00 mm
- net N$33: track 3.34 -> 0.00 mm
- net N$32: track 3.34 -> 0.00 mm
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Other:
- board size 46.4 x 293.7 mm -> 79.5 x 78 mm
- board text removed: "Common"
- board text removed: "Powered"
- board text removed: "Unpowered"
