File: Eagle/Computer Power Relay/Computer Power Relay - Merge.sch (EAGLE design)
At the start: 141 parts, among them K1 RELAY-3V3DC-110VAC012, K2 RELAY-110VACV3_IN-PLACE, U1 RP2040, U2 AP2112M-3.3TRG1, U3 SWITCH-SLIDE-DPDT, U4 SWITCH-SLIDE-DPDT, U5 SWITCH-SLIDE-DPDT, U6 RP2040, U7 AP2112M-3.3TRG1

Commit message: CPR 100% Complete
Damn shipping's expensive.  Better work on the other projects so I can subsidize this.
Parts:
- removed C18, C20, C22, C23, C46, C47, C48, C49, C51, C52, C53, C56, C57: 100nF, adafruit:CAP-NONPOL-USC0402K
- removed C19, C21, C24, C25: 47uF, adafruit:CAP-NONPOL-USC0402K
- removed C26, C27, C28, C29, C30, C31, C32, C33, C34, C35, C36, C37, C38, C39, C40, C41: (no value), Inventory:CAPACITOR-NONPOLARIZED
- removed C42, C43: (no value), adafruit:CAP-NONPOL-USC0402K
- removed C44, C45: ~30pF, adafruit:CAP-NONPOL-USC0402K
- removed C50, C55: 1uF, adafruit:CAP-NONPOL-USC0402K
- removed CLOCK1: 12MHz, crystal:CRYSTALHC49S
- removed COMPARATOR: COMPARATOR_LM393N, Inventory:COMPARATOR_LM393N
- removed DIGITAL, GROUND, PWM-1-OUT, PWM-2-OUT, PWM-OUT, R1-POLE1, R1-POLE2, R2-POLE1, R2-POLE2, R3-POLE1, R3-POLE2: (no value), adafruit:PINHD-1X1
- removed OP-AMP: OP-AMP_TDA2822N, Inventory:OP-AMP_TDA2822N
- removed POWER_SWITCH1: SWITCH-SLIDE-2P2T, Inventory:SWITCH-SLIDE-2P2T
- removed PWM1, PWM2, SV2: (no value), con-lstb:MA04-1
- removed R11, R14, R17, R18: 220 Ω, rcl:R-US_R0603
- removed R12, R15, R21, R22: 100 Ω, rcl:R-US_R0603
- removed R13, R16, R19, R20: 1.8K Ω, rcl:R-US_R0603
- removed R23, R25, R32, R33: (no value), rcl:R-US_R0603
- removed R24, R30, R31: 1MΩ, Inventory:POTENTIOMETER_3-PINPT-10
- removed R26, R29, R34: 10KΩ, Inventory:POTENTIOMETER_3-PINPT-10
- removed R27, R28, R35: 100Ω, Inventory:POTENTIOMETER_3-PINPT-10
- removed R36, R37: 27.4 Ω, rcl:R-US_R0603
- removed R38, R40: 1k Ω, rcl:R-US_R0603
- removed R39, R41: 10k Ω, rcl:R-US_R0603
- removed R43: 4.7k Ω, rcl:R-US_R0603
- removed SV1: (no value), con-lstb:MA03-1
- removed SW2: (no value), KVM Keyboard:SWITCH_PUSHBUTTONSOFTTOUCHSMD_SJ
- removed U$6: AUDIO_JACK_FEMALE_5-PIN, Inventory:AUDIO_JACK_FEMALE_5-PIN
- removed U$8: W25Q128JVSIM-ND__QSPI-FLASH, KVM Keyboard:W25Q128JVSIM-ND__QSPI-FLASH
- removed U3, U4, U5: SWITCH-SLIDE-DPDT, Inventory:SWITCH-SLIDE-DPDT
- removed U6: RP2040, KVM Keyboard:RP2040
- removed U7: AP2112M-3.3TRG1, KVM Keyboard:AP2112M-3.3TRG1
Connections:
- removed net 5V_2: POWER_SWITCH1.O, SV2.1, U7.VIN
- removed net D+_2: R36.2, SV2.3
- removed net D-_2: R37.2, SV2.2
- removed net DIGITAL: COMPARATORB.+IN, COMPARATORG$1.OUT, SV1.2
- removed net GND-3: C18.2, PWM1.1, R12.2, R13.2
- removed net GND-4: C20.2, C22.2, C23.2, PWM2.1, R15.2, R16.2
- removed net GND-5: C26.2, C35.2, C36.2, C37.2, C38.2, C39.2, C40.2, C41.2, GROUND.1, U4.4, U5.3
- removed net GND-6: C43.2, COMPARATORB.-IN, COMPARATORG$1.-IN, R32.1, U$6.GND
- removed net GND-7: POWER_SWITCH1.S, SV2.4, U7.GND, U7.GND_2
- removed net N$10: C19.1, PWM-1-OUT.1, R13.1
- removed net N$11: C20.1, C21.2, C22.1, C23.1, C24.2, C25.2, R14.1, R22.1
- removed net N$12: C21.1, C24.1, C25.1, PWM-2-OUT.1, R20.1
- removed net N$13: R17.1, R18.1
- removed net N$14: R14.2, R17.2
- removed net N$15: R19.2, R20.2
- removed net N$21: R16.1, R19.1
- removed net N$22: R15.1, R21.1
- removed net N$23: R21.2, R22.2
- removed net N$24: DIGITAL.1, U3.3
- removed net N$25: R24.2, R24.3, R26.1
- removed net N$26: C27.1, C28.1, C29.1, C30.1, C31.1, C32.1, C33.1, C34.1, PWM-OUT.1, U5.4
- removed net N$27: R26.2, R26.3, R27.1
- removed net N$28: R27.2, R27.3, U3.5
- removed net N$29: R24.1, U3.2
- removed net N$30: R1-POLE1.1, U3.1
- removed net N$31: R1-POLE2.1, U3.6
- removed net N$32: R2-POLE2.1, U4.6
- removed net N$33: R2-POLE1.1, U4.1
- removed net N$34: R30.1, U4.2
- removed net N$35: R28.2, R28.3, U4.5
- removed net N$36: R3-POLE2.1, U5.6
- removed net N$37: R3-POLE1.1, U5.1
- removed net N$38: R28.1, R29.2, R29.3
- removed net N$39: R29.1, R30.2, R30.3
- removed net N$40: R31.1, U5.2
- removed net N$41: R34.2, R34.3, R35.1
- removed net N$42: R31.2, R31.3, R34.1
- removed net N$43: R35.2, R35.3, U5.5
- removed net N$44: C26.1, C27.2, C28.2, C29.2, C30.2, C31.2, C32.2, C33.2, C34.2, C35.1, C36.1, C37.1, C38.1, C39.1, C40.1, C41.1, U3.4, U4.3
- removed net N$45: OP-AMPG$1.+IN, U$6.LEFT, U$6.LTEST
- removed net N$46: R36.1, U6.USB_DP
- removed net N$47: OP-AMPB.+IN, R32.2
- removed net N$51: C43.1, OP-AMPG$1.-IN, R33.2
- removed net N$52: OP-AMPG$1.OUT, R23.1
- removed net N$53: C42.1, OP-AMPB.-IN, R23.2, R25.1
- removed net N$54: C42.2, COMPARATORG$1.+IN, OP-AMPB.OUT, R25.2
- removed net N$55: R37.1, U6.USB_DM
- removed net N$56: COMPARATORB.OUT, R33.1
- removed net N$57: C45.2, CLOCK1.2, R38.1
- removed net N$58: R38.2, U6.XOUT
- removed net N$59: C44.2, CLOCK1.1, U6.XIN
- removed net N$6: PWM1.2, PWM1.3, PWM1.4, R11.2
- removed net N$60: U$8.IO2, U6.QSPI_SD2
- removed net N$61: U$8.IO1, U6.QSPI_SD1
- removed net N$62: U$8.IO0, U6.QSPI_SD0
- removed net N$63: U$8.CLK, U6.QSPI_SCLK
- removed net N$64: U$8.IO3, U6.QSPI_SD3
- removed net N$7: C18.1, C19.2, R11.1, R12.1
- removed net N$8: PWM2.2, PWM2.3, PWM2.4, R18.2
- removed net SD-V+: COMPARATORG$1.V+, OP-AMPG$1.V+, SV1.1
- removed net SD-V-: COMPARATORG$1.V-, OP-AMPG$1.V-, SV1.3
- net 1V1: no longer C55.2, C56.2, C57.2, U6.DVDD, U6.DVDD_2, U6.VREG_VOUT
- net 3V3: no longer C46.2, C47.2, C48.2, C49.2, C50.2, C51.2, C52.2, C53.2, R39.2, U$8.VCC, U6.ADC_AVDD, U6.IOVDD, U6.IOVDD_2, U6.IOVDD_3, U6.IOVDD_4, U6.IOVDD_5, U6.IOVDD_6, U6.USB_VDD, U6.VREG_VIN, U7.VOUT
- net BOOTSEL: no longer R40.2
- net BUTTON: no longer R43.1, SW2.P$1
- net EN: no longer R41.2, U7.EN
- net GND: no longer C44.1, C45.1, C46.1, C47.1, C48.1, C49.1, C50.1, C51.1, C52.1, C53.1, C55.1, C56.1, C57.1, SW2.P$2, U$8.GND, U6.GND, U6.TESTEN
- net QSPI_SS_N: no longer R39.1, R40.1, U$8./CS, U6.QSPI_SS_N
- net RUN: no longer R43.2, U6.RUN
- net SWITCH: no longer POWER_SWITCH1.P, R41.1
Other:
- moved on the sheet: K1, K2

Commit message: (CPR) 90% done, almost ready to send to fab
Power Strip board is 100% complete.
Controller board is 95% complete, all that's left is to figure out a method to restart into Boot Select with a single button press, and double-check that it works before sending it off to print.

Remaining space of board is being filled out, and is nearly finished.

I'm considering adding plated holes for spacer holes into the Power Strip board.  We'll see.
Parts:
- added C18, C20, C22, C23, C46, C47, C48, C49, C51, C52, C53, C56, C57: 100nF, adafruit:CAP-NONPOL-USC0402K
- added C19, C21, C24, C25: 47uF, adafruit:CAP-NONPOL-USC0402K
- added C26, C27, C28, C29, C30, C31, C32, C33, C34, C35, C36, C37, C38, C39, C40, C41: (no value), Inventory:CAPACITOR-NONPOLARIZED
- added C42, C43: (no value), adafruit:CAP-NONPOL-USC0402K
- added C44, C45: ~30pF, adafruit:CAP-NONPOL-USC0402K
- added C50, C55: 1uF, adafruit:CAP-NONPOL-USC0402K
- added CLOCK1: 12MHz, crystal:CRYSTALHC49S
- added COMPARATOR: COMPARATOR_LM393N, Inventory:COMPARATOR_LM393N
- added DIGITAL, GROUND, PWM-1-OUT, PWM-2-OUT, PWM-OUT, R1-POLE1, R1-POLE2, R2-POLE1, R2-POLE2, R3-POLE1, R3-POLE2: (no value), adafruit:PINHD-1X1
- added OP-AMP: OP-AMP_TDA2822N, Inventory:OP-AMP_TDA2822N
- added POWER_SWITCH1: SWITCH-SLIDE-2P2T, Inventory:SWITCH-SLIDE-2P2T
- added PWM1, PWM2, SV2: (no value), con-lstb:MA04-1
- added R11, R14, R17, R18: 220 Ω, rcl:R-US_R0603
- added R12, R15, R21, R22: 100 Ω, rcl:R-US_R0603
- added R13, R16, R19, R20: 1.8K Ω, rcl:R-US_R0603
- added R23, R25, R32, R33: (no value), rcl:R-US_R0603
- added R24, R30, R31: 1MΩ, Inventory:POTENTIOMETER_3-PINPT-10
- added R26, R29, R34: 10KΩ, Inventory:POTENTIOMETER_3-PINPT-10
- added R27, R28, R35: 100Ω, Inventory:POTENTIOMETER_3-PINPT-10
- added R36, R37: 27.4 Ω, rcl:R-US_R0603
- added R38, R40: 1k Ω, rcl:R-US_R0603
- added R39, R41: 10k Ω, rcl:R-US_R0603
- added R43: 4.7k Ω, rcl:R-US_R0603
- added SV1: (no value), con-lstb:MA03-1
- added SW2: (no value), KVM Keyboard:SWITCH_PUSHBUTTONSOFTTOUCHSMD_SJ
- added U$6: AUDIO_JACK_FEMALE_5-PIN, Inventory:AUDIO_JACK_FEMALE_5-PIN
- added U$8: W25Q128JVSIM-ND__QSPI-FLASH, KVM Keyboard:W25Q128JVSIM-ND__QSPI-FLASH
- added U3, U4, U5: SWITCH-SLIDE-DPDT, Inventory:SWITCH-SLIDE-DPDT
- added U6: RP2040, KVM Keyboard:RP2040
- added U7: AP2112M-3.3TRG1, KVM Keyboard:AP2112M-3.3TRG1
Connections:
- new net 5V_2: POWER_SWITCH1.O, SV2.1, U7.VIN
- new net D+_2: R36.2, SV2.3
- new net D-_2: R37.2, SV2.2
- new net DIGITAL: COMPARATORB.+IN, COMPARATORG$1.OUT, SV1.2
- new net GND-3: C18.2, PWM1.1, R12.2, R13.2
- new net GND-4: C20.2, C22.2, C23.2, PWM2.1, R15.2, R16.2
- new net GND-5: C26.2, C35.2, C36.2, C37.2, C38.2, C39.2, C40.2, C41.2, GROUND.1, U4.4, U5.3
- new net GND-6: C43.2, COMPARATORB.-IN, COMPARATORG$1.-IN, R32.1, U$6.GND
- new net GND-7: POWER_SWITCH1.S, SV2.4, U7.GND, U7.GND_2
- new net N$10: C19.1, PWM-1-OUT.1, R13.1
- new net N$11: C20.1, C21.2, C22.1, C23.1, C24.2, C25.2, R14.1, R22.1
- new net N$12: C21.1, C24.1, C25.1, PWM-2-OUT.1, R20.1
- new net N$13: R17.1, R18.1
- new net N$14: R14.2, R17.2
- new net N$15: R19.2, R20.2
- new net N$21: R16.1, R19.1
- new net N$22: R15.1, R21.1
- new net N$23: R21.2, R22.2
- new net N$24: DIGITAL.1, U3.3
- new net N$25: R24.2, R24.3, R26.1
- new net N$26: C27.1, C28.1, C29.1, C30.1, C31.1, C32.1, C33.1, C34.1, PWM-OUT.1, U5.4
- new net N$27: R26.2, R26.3, R27.1
- new net N$28: R27.2, R27.3, U3.5
- new net N$29: R24.1, U3.2
- new net N$30: R1-POLE1.1, U3.1
- new net N$31: R1-POLE2.1, U3.6
- new net N$32: R2-POLE2.1, U4.6
- new net N$33: R2-POLE1.1, U4.1
- new net N$34: R30.1, U4.2
- new net N$35: R28.2, R28.3, U4.5
- new net N$36: R3-POLE2.1, U5.6
- new net N$37: R3-POLE1.1, U5.1
- new net N$38: R28.1, R29.2, R29.3
- new net N$39: R29.1, R30.2, R30.3
- new net N$40: R31.1, U5.2
- new net N$41: R34.2, R34.3, R35.1
- new net N$42: R31.2, R31.3, R34.1
- new net N$43: R35.2, R35.3, U5.5
- new net N$44: C26.1, C27.2, C28.2, C29.2, C30.2, C31.2, C32.2, C33.2, C34.2, C35.1, C36.1, C37.1, C38.1, C39.1, C40.1, C41.1, U3.4, U4.3
- new net N$45: OP-AMPG$1.+IN, U$6.LEFT, U$6.LTEST
- new net N$46: R36.1, U6.USB_DP
- new net N$47: OP-AMPB.+IN, R32.2
- new net N$51: C43.1, OP-AMPG$1.-IN, R33.2
- new net N$52: OP-AMPG$1.OUT, R23.1
- new net N$53: C42.1, OP-AMPB.-IN, R23.2, R25.1
- new net N$54: C42.2, COMPARATORG$1.+IN, OP-AMPB.OUT, R25.2
- new net N$55: R37.1, U6.USB_DM
- new net N$56: COMPARATORB.OUT, R33.1
- new net N$57: C45.2, CLOCK1.2, R38.1
- new net N$58: R38.2, U6.XOUT
- new net N$59: C44.2, CLOCK1.1, U6.XIN
- new net N$6: PWM1.2, PWM1.3, PWM1.4, R11.2
- new net N$60: U$8.IO2, U6.QSPI_SD2
- new net N$61: U$8.IO1, U6.QSPI_SD1
- new net N$62: U$8.IO0, U6.QSPI_SD0
- new net N$63: U$8.CLK, U6.QSPI_SCLK
- new net N$64: U$8.IO3, U6.QSPI_SD3
- new net N$7: C18.1, C19.2, R11.1, R12.1
- new net N$8: PWM2.2, PWM2.3, PWM2.4, R18.2
- new net SD-V+: COMPARATORG$1.V+, OP-AMPG$1.V+, SV1.1
- new net SD-V-: COMPARATORG$1.V-, OP-AMPG$1.V-, SV1.3
- net 1V1: now also C55.2, C56.2, C57.2, U6.DVDD, U6.DVDD_2, U6.VREG_VOUT
- net 3V3: now also C46.2, C47.2, C48.2, C49.2, C50.2, C51.2, C52.2, C53.2, R39.2, U$8.VCC, U6.ADC_AVDD, U6.IOVDD, U6.IOVDD_2, U6.IOVDD_3, U6.IOVDD_4, U6.IOVDD_5, U6.IOVDD_6, U6.USB_VDD, U6.VREG_VIN, U7.VOUT
- net BOOTSEL: now also R40.2
- net BUTTON: now also R43.1, SW2.P$1
- net EN: now also R41.2, U7.EN
- net GND: now also C44.1, C45.1, C46.1, C47.1, C48.1, C49.1, C50.1, C51.1, C52.1, C53.1, C55.1, C56.1, C57.1, SW2.P$2, U$8.GND, U6.GND, U6.TESTEN
- net QSPI_SS_N: now also R39.1, R40.1, U$8./CS, U6.QSPI_SS_N
- net RUN: now also R43.2, U6.RUN
- net SWITCH: now also POWER_SWITCH1.P, R41.1
Other:
- moved on the sheet: K1, K2
