File: Eagle/KVM-Keyboard/KVM Keyboard.brd (EAGLE design)
At the start: 460.8 x 147.5 mm, 284 parts

Commit message: Edited libraries & added USBs
I edited library symbols to be more clear in the schematic about what they actually are.  They should be much easier to understand than plain rectangles.

I began adding USB ports, USB hub, and some RP2040s.

When I left off, I was trying to redraw the symbol for a 2:2 mux for swapping between USB signals.
Parts:
- added D1, D10, D11, D12, D2, D3, D4, D5, D6, D7, D8, D9: (no value), KVM-Keyboard:DIODE_SMALL
- added U$1: USB.HUB-USB3.1-6.PORT__USB7206C/KDXVQFN100_KDX_MCH, KVM-Keyboard:VQFN100_KDX_MCH
- added U$2, U$3, U$4, U$5, U$6: QSPI-FLASH__W25Q128JVSIM-ND, KVM-Keyboard:SO08
- added U1, U2, U3, U4, U5: RP2040, KVM-Keyboard:IC57_RP2040
- added USB1, USB2, USB3, USB4, USB5, USB6: USB-C_RECEPTACLE, KVM-Keyboard:USB-C_RECEPTACLE
Connections:
- new net 18.VCORE: U$1.18
- new net 25.VCORE: U$1.25
- new net 26.VDD33: U$1.26
- new net 31.VCORE: U$1.31
- new net 38.VCORE: U$1.38
- new net 43.VDD33: U$1.43
- new net 53.VDD33: U$1.53
- new net 55.VCORE: U$1.55
- new net 62.VDD33: U$1.62
- new net 67.VDD33: U$1.67
- new net 78.VCORE: U$1.78
- new net 79.VDD33: U$1.79
- new net 85.VCORE: U$1.85
- new net 88.VDD33: U$1.88
- new net 9.VCORE: U$1.9
- new net 93.VCORE: U$1.93
- new net 99.VDD33: U$1.99
- new net ADC_AVDD: U1.43, U2.43, U3.43, U4.43, U5.43
- new net DVDD: U1.50, U2.50, U3.50, U4.50, U5.50
- new net DVDD_2: U1.23, U2.23, U3.23, U4.23, U5.23
- new net GND: D1.A, D10.A, D11.A, D3.A, D6.A, D7.A, U$1.101
- new net IOVDD: U1.49, U2.49, U3.49, U4.49, U5.49
- new net IOVDD_2: U1.1, U2.1, U3.1, U4.1, U5.1
- new net IOVDD_3: U1.10, U2.10, U3.10, U4.10, U5.10
- new net IOVDD_4: U1.22, U2.22, U3.22, U4.22, U5.22
- new net IOVDD_5: U1.33, U2.33, U3.33, U4.33, U5.33
- new net IOVDD_6: U1.42, U2.42, U3.42, U4.42, U5.42
- new net N$1: U$2.1, U1.56
- new net N$10: U$3.5, U2.53
- new net N$11: U$3.3, U2.54
- new net N$12: U$3.2, U2.55
- new net N$13: U$4.1, U3.56
- new net N$14: U$4.7, U3.51
- new net N$15: U$4.6, U3.52
- new net N$16: U$4.5, U3.53
- new net N$17: U$4.3, U3.54
- new net N$18: U$4.2, U3.55
- new net N$19: U$5.1, U4.56
- new net N$2: U$2.6, U1.52
- new net N$20: U$5.7, U4.51
- new net N$21: U$5.6, U4.52
- new net N$22: U$5.5, U4.53
- new net N$23: U$5.3, U4.54
- new net N$24: U$5.2, U4.55
- new net N$25: U$6.1, U5.56
- new net N$26: U$6.7, U5.51
- new net N$27: U$6.6, U5.52
- new net N$28: U$6.5, U5.53
- new net N$29: U$6.3, U5.54
- new net N$3: U$2.5, U1.53
- new net N$30: U$6.2, U5.55
- new net N$4: U$2.2, U1.55
- new net N$5: U$2.3, U1.54
- new net N$6: U$2.7, U1.51
- new net N$7: U$3.1, U2.56
- new net N$8: U$3.7, U2.51
- new net N$9: U$3.6, U2.52
- new net PICO.D+: U$1.42, U5.47
- new net PICO.D-: U$1.41, U5.46
- new net USB.SHIELDING: USB1.25, USB1.26, USB1.27, USB1.28, USB2.25, USB2.26, USB2.27, USB2.28, USB3.25, USB3.26, USB3.27, USB3.28, USB4.25, USB4.26, USB4.27, USB4.28, USB5.25, USB5.26, USB5.27, USB5.28, USB6.25, USB6.26, USB6.27, USB6.28
- new net USB1.CC1: USB1.A5
- new net USB1.CC2: USB1.B5
- new net USB1.D+: USB1.A6, USB1.B6
- new net USB1.D-: USB1.A7, USB1.B7
- new net USB1.GND: D1.C, USB1.A1, USB1.A12, USB1.B1, USB1.B12
- new net USB1.R+: U$1.94, USB1.B11
- new net USB1.RX+: USB1.A11
- new net USB1.RX-: USB1.A10
- new net USB1.SBU: USB1.A8, USB1.B8, USB1.B9
- new net USB1.TX+: U$1.91, USB1.A2, USB1.B2
- new net USB1.TX-: U$1.92, USB1.A3, USB1.B3
- new net USB1.VBUS: D2.A, USB1.A4, USB1.A9, USB1.B4
- new net USB1RX-: U$1.95, USB1.B10
- new net USB2.CC1: USB2.A5
- new net USB2.CC2: USB2.B5
- new net USB2.D+: USB2.A6, USB2.B6
- new net USB2.D-: USB2.A7, USB2.B7
- new net USB2.GND: D3.C, USB2.A1, USB2.A12, USB2.B1, USB2.B12
- new net USB2.RX+: U$1.10, USB2.A11, USB2.B11
- new net USB2.RX-: U$1.11, USB2.A10, USB2.B10
- new net USB2.SBU: USB2.A8, USB2.B8
- new net USB2.TX+: U$1.7, USB2.A2, USB2.B2
- new net USB2.TX-: U$1.8, USB2.A3, USB2.B3
- new net USB2.VBUS: D4.A, USB2.A4, USB2.A9, USB2.B4, USB2.B9
- new net USB3.CC1: USB3.A5
- new net USB3.CC2: USB3.B5
- new net USB3.D+: USB3.A6, USB3.B6
- new net USB3.D-: USB3.A7, USB3.B7
- new net USB3.GND: D6.C, USB3.A1, USB3.A12, USB3.B1, USB3.B12
- new net USB3.RX+: U$1.19, USB3.A11, USB3.B11
- new net USB3.RX-: U$1.20, USB3.A10, USB3.B10
- new net USB3.SBU: USB3.A8, USB3.B8
- new net USB3.TX+: U$1.16, USB3.A2, USB3.B2
- new net USB3.TX-: U$1.17, USB3.A3, USB3.B3
- new net USB3.VBUS: D5.A, USB3.A4, USB3.A9, USB3.B4, USB3.B9
- new net USB4.CC1: USB4.A5
- new net USB4.CC2: USB4.B5
- new net USB4.D+: USB4.A6, USB4.B6
- new net USB4.D-: USB4.A7, USB4.B7
- new net USB4.GND: D7.C, USB4.A1, USB4.A12, USB4.B1, USB4.B12
- new net USB4.RX+: U$1.32, USB4.A11, USB4.B11
- new net USB4.RX-: U$1.33, USB4.A10, USB4.B10
- new net USB4.SBU: USB4.A8, USB4.B8
- new net USB4.TX+: U$1.29, USB4.A2, USB4.B2
- new net USB4.TX-: U$1.30, USB4.A3, USB4.B3
- new net USB4.VBUS: D8.A, USB4.A4, USB4.A9, USB4.B4, USB4.B9
- new net USB5.CC1: USB5.A5
- new net USB5.CC2: USB5.B5
- new net USB5.D+: U$1.34, USB5.A6, USB5.B6
- new net USB5.D-: U$1.35, USB5.A7, USB5.B7
- new net USB5.GND: D10.C, USB5.A1, USB5.A12, USB5.B1, USB5.B12
- new net USB5.RX+: U$1.39, USB5.A11, USB5.B11
- new net USB5.RX-: U$1.40, USB5.A10, USB5.B10
- new net USB5.SBU: USB5.A8, USB5.B8
- new net USB5.TX+: U$1.36, USB5.A2, USB5.B2
- new net USB5.TX-: U$1.37, USB5.A3, USB5.B3
- new net USB5.VBUS: D9.A, USB5.A4, USB5.A9, USB5.B4, USB5.B9
- new net USB6.CC1: USB6.A5
- new net USB6.CC2: USB6.B5
- new net USB6.D+: U$1.81, USB6.A6, USB6.B6
- new net USB6.D-: U$1.82, USB6.A7, USB6.B7
- new net USB6.GND: D11.C, USB6.A1, USB6.A12, USB6.B1, USB6.B12
- new net USB6.RX+: U$1.86, USB6.A11, USB6.B11
- new net USB6.RX-: U$1.87, USB6.A10, USB6.B10
- new net USB6.SBU: USB6.A8, USB6.B8
- new net USB6.TX+: U$1.83, USB6.A2, USB6.B2
- new net USB6.TX-: U$1.84, USB6.A3, USB6.B3
- new net USB6.VBUS: D12.A, USB6.A4, USB6.A9, USB6.B4, USB6.B9
- new net USB_VDD: U1.48, U2.48, U3.48, U4.48, U5.48
- new net VCC: D12.C, D2.C, D4.C, D5.C, D8.C, D9.C

Commit message: Small update
Parts:
- added U6, U7: MUX.DEMUX-8X.2:2_PI3PCIE3242AZLEX, KVM-Keyboard:30-WFQFN_EXPOSED.PAD
Connections:
- new net 13.GND: U6.13, U7.13
- new net OE#: U6.29, U7.29
- new net SEL: U6.5, U7.5
Changed lines of the file:
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@@
 <attribute name="VALUE" x="-270.75" y="-239.2" size="1.27" layer="27" ratio="10" align="center"/>
+</element>
+<element name="U6" library="KVM-Keyboard" package="30-WFQFN_EXPOSED.PAD" value="MUX.DEMUX-8X.2:2_PI3PCIE3242AZLEX" x="-270.75" y="-247" smashed="yes">
+<attribute name="COPYRIGHT" value="Copyright (C) 2022 Ultra Librarian. All rights reserved." x="-270.75" y="-247" size="1.778" layer="27" display="off"/>
+<attribute name="MANUFACTURER_PART_NUMBER" value="HD3SS3220IRNHR" x="-270.75" y="-247" size="1.778" layer="27" display="off"/>
+<attribute name="MFR_NAME" value="Texas Instruments" x="-270.75" y="-247" size="1.778" layer="27" display="off"/>
+<attribute name="NAME" x="-274.0266" y="-247.635" size="1.27" layer="27" ratio="6" rot="SR0" align="center-left"/>
+<attribute name="REFDES" value="RefDes" x="-270.75" y="-247" size="1.778" layer="27" display="off"/>
+<attribute name="TYPE" value="TYPE" x="-270.75" y="-247" size="1.778" layer="27" display="off"/>
+<attribute name="VALUE" x="-272.4772" y="-247.635" size="1.27" layer="21" ratio="6" rot="SR0" align="center-left"/>
+</element>
+<element name="U7" library="KVM-Keyboard" package="30-WFQFN_EXPOSED.PAD" value="MUX.DEMUX-8X.2:2_PI3PCIE3242AZLEX" x="-270.75" y="-256.5" smashed="yes">
+<attribute name="COPYRIGHT" value="Copyright (C) 2022 Ultra Librarian. All rights reserved." x="-270.75" y="-256.5" size="1.778" layer="27" display="off"/>
+<attribute name="MANUFACTURER_PART_NUMBER" value="HD3SS3220IRNHR" x="-270.75" y="-256.5" size="1.778" layer="27" display="off"/>
+<attribute name="MFR_NAME" value="Texas Instruments" x="-270.75" y="-256.5" size="1.778" layer="27" display="off"/>
+<attribute name="NAME" x="-274.0266" y="-257.135" size="1.27" layer="27" ratio="6" rot="SR0" align="center-left"/>
+<attribute name="REFDES" value="RefDes" x="-270.75" y="-256.5" size="1.778" layer="27" display="off"/>
+<attribute name="TYPE" value="TYPE" x="-270.75" y="-256.5" size="1.778" layer="27" display="off"/>
+<attribute name="VALUE" x="-272.4772" y="-257.135" size="1.27" layer="21" ratio="6" rot="SR0" align="center-left"/>
 </element>
 </elements>
@@
 <wire x1="-273.29" y1="-237.5" x2="-273.29" y2="-223.25" width="0" layer="19" extent="1-1"/>
 </signal>
+<signal name="SEL">
+<contactref element="U6" pad="5"/>
+<contactref element="U7" pad="5"/>
+<wire x1="-271.95" y1="-246.8" x2="-271.95" y2="-256.3" width="0" layer="19" extent="1-1"/>
+</signal>
+<signal name="13.GND">
+<contactref element="U6" pad="13"/>
+<contactref element="U7" pad="13"/>
+<wire x1="-270.75" y1="-249.199996875" x2="-270.75" y2="-258.699996875" width="0" layer="19" extent="1-1"/>
+</signal>
+<signal name="OE#">
+<contactref element="U6" pad="29"/>
+<contactref element="U7" pad="29"/>
+<wire x1="-271.15" y1="-244.8" x2="-271.15" y2="-254.3" width="0" layer="19" extent="1-1"/>
+</signal>
 </signals>

Commit message: Begun Neopixel testing
Connections:
- net PICO.D+: no longer U$1.42
- net PICO.D-: no longer U$1.41
- net USB1.R+: no longer U$1.94
- net USB1.TX+: no longer U$1.91
- net USB1.TX-: no longer U$1.92
- net USB1RX-: no longer U$1.95
- net USB2.RX+: no longer U$1.10
- net USB2.RX-: no longer U$1.11
- net USB2.TX+: no longer U$1.7
- net USB2.TX-: no longer U$1.8
- net USB3.RX+: no longer U$1.19
- net USB3.RX-: no longer U$1.20
- net USB3.TX+: no longer U$1.16
- net USB3.TX-: no longer U$1.17
- net USB4.RX+: no longer U$1.32
- net USB4.RX-: no longer U$1.33
- net USB4.TX+: no longer U$1.29
- net USB4.TX-: no longer U$1.30
- net USB5.D+: no longer U$1.34
- net USB5.D-: no longer U$1.35
- net USB5.RX+: no longer U$1.39
- net USB5.RX-: no longer U$1.40
- net USB5.TX+: no longer U$1.36
- net USB5.TX-: no longer U$1.37
- net USB6.D+: no longer U$1.81
- net USB6.D-: no longer U$1.82
- net USB6.RX+: no longer U$1.86
- net USB6.RX-: no longer U$1.87
- net USB6.TX+: no longer U$1.83
- net USB6.TX-: no longer U$1.84
