File: Eagle/KVM-Keyboard/KVM Keyboard.sch (EAGLE design)
At the start: 284 parts

Commit message: Edited libraries & added USBs
I edited library symbols to be more clear in the schematic about what they actually are.  They should be much easier to understand than plain rectangles.

I began adding USB ports, USB hub, and some RP2040s.

When I left off, I was trying to redraw the symbol for a 2:2 mux for swapping between USB signals.
Parts:
- added D1, D10, D11, D12, D2, D3, D4, D5, D6, D7, D8, D9: (no value), KVM-Keyboard:DIODESMALL
- added U$1: USB.HUB-USB3.1-6.PORT__USB7206C/KDXVQFN100_KDX_MCH, KVM-Keyboard:USB.HUB-USB3.1-6.PORT__USB7206C/KDXVQFN100_KDX_MCH
- added U$2, U$3, U$4, U$5, U$6: QSPI-FLASH__W25Q128JVSIM-ND, KVM-Keyboard:QSPI-FLASH__W25Q128JVSIM-ND
- added U1, U2, U3, U4, U5: RP2040, KVM-Keyboard:RP2040
- added USB1, USB2, USB3, USB4, USB5, USB6: USB-C_RECEPTACLE, KVM-Keyboard:USB-C_RECEPTACLE
Connections:
- new net GND: D1.A, D10.A, D11.A, D3.A, D6.A, D7.A, U$1.101.VSS
- new net N$1: U$2./CS, U1.QSPI_SS_N
- new net N$10: U$3.IO0(DI), U2.QSPI_SD0
- new net N$11: U$3.IO2(/WP), U2.QSPI_SD2
- new net N$12: U$3.IO1(DO), U2.QSPI_SD1
- new net N$13: U$4./CS, U3.QSPI_SS_N
- new net N$14: U$4.IO3, U3.QSPI_SD3
- new net N$15: U$4.CLK, U3.QSPI_SCLK
- new net N$16: U$4.IO0(DI), U3.QSPI_SD0
- new net N$17: U$4.IO2(/WP), U3.QSPI_SD2
- new net N$18: U$4.IO1(DO), U3.QSPI_SD1
- new net N$19: U$5./CS, U4.QSPI_SS_N
- new net N$2: U$2.CLK, U1.QSPI_SCLK
- new net N$20: U$5.IO3, U4.QSPI_SD3
- new net N$21: U$5.CLK, U4.QSPI_SCLK
- new net N$22: U$5.IO0(DI), U4.QSPI_SD0
- new net N$23: U$5.IO2(/WP), U4.QSPI_SD2
- new net N$24: U$5.IO1(DO), U4.QSPI_SD1
- new net N$25: U$6./CS, U5.QSPI_SS_N
- new net N$26: U$6.IO3, U5.QSPI_SD3
- new net N$27: U$6.CLK, U5.QSPI_SCLK
- new net N$28: U$6.IO0(DI), U5.QSPI_SD0
- new net N$29: U$6.IO2(/WP), U5.QSPI_SD2
- new net N$3: U$2.IO0(DI), U1.QSPI_SD0
- new net N$30: U$6.IO1(DO), U5.QSPI_SD1
- new net N$4: U$2.IO1(DO), U1.QSPI_SD1
- new net N$5: U$2.IO2(/WP), U1.QSPI_SD2
- new net N$6: U$2.IO3, U1.QSPI_SD3
- new net N$7: U$3./CS, U2.QSPI_SS_N
- new net N$8: U$3.IO3, U2.QSPI_SD3
- new net N$9: U$3.CLK, U2.QSPI_SCLK
- new net PICO.D+: U$1.42.USB2DN_DP6/PRT_DIS_P6, U5.USB_DP
- new net PICO.D-: U$1.41.USB2DN_DM6/PRT_DIS_M6, U5.USB_DM
- new net USB.SHIELDING: USB1.SHIELDING, USB2.SHIELDING, USB3.SHIELDING, USB4.SHIELDING, USB5.SHIELDING, USB6.SHIELDING
- new net USB1.CC1: USB1.A5
- new net USB1.CC2: USB1.B5
- new net USB1.D+: USB1.A6, USB1.B6
- new net USB1.D-: USB1.A7, USB1.B7
- new net USB1.GND: D1.C, USB1.A1, USB1.A12, USB1.B1, USB1.B12
- new net USB1.R+: U$1.94.USB3UP_RXDP, USB1.B11
- new net USB1.RX+: USB1.A11
- new net USB1.RX-: USB1.A10
- new net USB1.SBU: USB1.A8, USB1.B8, USB1.B9
- new net USB1.TX+: U$1.91.USB3UP_TXDP, USB1.A2, USB1.B2
- new net USB1.TX-: U$1.92.USB3UP_TXDM, USB1.A3, USB1.B3
- new net USB1.VBUS: D2.A, USB1.A4, USB1.A9, USB1.B4
- new net USB1RX-: U$1.95.USB3UP_RXDM, USB1.B10
- new net USB2.CC1: USB2.A5
- new net USB2.CC2: USB2.B5
- new net USB2.D+: USB2.A6, USB2.B6
- new net USB2.D-: USB2.A7, USB2.B7
- new net USB2.GND: D3.C, USB2.A1, USB2.A12, USB2.B1, USB2.B12
- new net USB2.RX+: U$1.10.USB3DN_RXDP1, USB2.A11, USB2.B11
- new net USB2.RX-: U$1.11.USB3DN_RXDM1, USB2.A10, USB2.B10
- new net USB2.SBU: USB2.A8, USB2.B8
- new net USB2.TX+: U$1.7.USB3DN_TXDP1, USB2.A2, USB2.B2
- new net USB2.TX-: U$1.8.USB3DN_TXDM1, USB2.A3, USB2.B3
- new net USB2.VBUS: D4.A, USB2.A4, USB2.A9, USB2.B4, USB2.B9
- new net USB3.CC1: USB3.A5
- new net USB3.CC2: USB3.B5
- new net USB3.D+: USB3.A6, USB3.B6
- new net USB3.D-: USB3.A7, USB3.B7
- new net USB3.GND: D6.C, USB3.A1, USB3.A12, USB3.B1, USB3.B12
- new net USB3.RX+: U$1.19.USB3DN_RXDP2, USB3.A11, USB3.B11
- new net USB3.RX-: U$1.20.USB3DN_RXDM2, USB3.A10, USB3.B10
- new net USB3.SBU: USB3.A8, USB3.B8
- new net USB3.TX+: U$1.16.USB3DN_TXDP2, USB3.A2, USB3.B2
- new net USB3.TX-: U$1.17.USB3DN_TXDM2, USB3.A3, USB3.B3
- new net USB3.VBUS: D5.A, USB3.A4, USB3.A9, USB3.B4, USB3.B9
- new net USB4.CC1: USB4.A5
- new net USB4.CC2: USB4.B5
- new net USB4.D+: USB4.A6, USB4.B6
- new net USB4.D-: USB4.A7, USB4.B7
- new net USB4.GND: D7.C, USB4.A1, USB4.A12, USB4.B1, USB4.B12
- new net USB4.RX+: U$1.32.USB3DN_RXDP3, USB4.A11, USB4.B11
- new net USB4.RX-: U$1.33.USB3DN_RXDM3, USB4.A10, USB4.B10
- new net USB4.SBU: USB4.A8, USB4.B8
- new net USB4.TX+: U$1.29.USB3DN_TXDP3, USB4.A2, USB4.B2
- new net USB4.TX-: U$1.30.USB3DN_TXDM3, USB4.A3, USB4.B3
- new net USB4.VBUS: D8.A, USB4.A4, USB4.A9, USB4.B4, USB4.B9
- new net USB5.CC1: USB5.A5
- new net USB5.CC2: USB5.B5
- new net USB5.D+: U$1.34.USB2DN_DP4/PRT_DIS_P4, USB5.A6, USB5.B6
- new net USB5.D-: U$1.35.USB2DN_DM4/PRT_DIS_M4, USB5.A7, USB5.B7
- new net USB5.GND: D10.C, USB5.A1, USB5.A12, USB5.B1, USB5.B12
- new net USB5.RX+: U$1.39.USB3DN_RXDP4, USB5.A11, USB5.B11
- new net USB5.RX-: U$1.40.USB3DN_RXDM4, USB5.A10, USB5.B10
- new net USB5.SBU: USB5.A8, USB5.B8
- new net USB5.TX+: U$1.36.USB3DN_TXDP4, USB5.A2, USB5.B2
- new net USB5.TX-: U$1.37.USB3DN_TXDM4, USB5.A3, USB5.B3
- new net USB5.VBUS: D9.A, USB5.A4, USB5.A9, USB5.B4, USB5.B9
- new net USB6.CC1: USB6.A5
- new net USB6.CC2: USB6.B5
- new net USB6.D+: U$1.81.USB2DN_DP5/PRT_DIS_P5, USB6.A6, USB6.B6
- new net USB6.D-: U$1.82.USB2DN_DM5/PRT_DIS_M5, USB6.A7, USB6.B7
- new net USB6.GND: D11.C, USB6.A1, USB6.A12, USB6.B1, USB6.B12
- new net USB6.RX+: U$1.86.USB3DN_RXDP5, USB6.A11, USB6.B11
- new net USB6.RX-: U$1.87.USB3DN_RXDM5, USB6.A10, USB6.B10
- new net USB6.SBU: USB6.A8, USB6.B8
- new net USB6.TX+: U$1.83.USB3DN_TXDP5, USB6.A2, USB6.B2
- new net USB6.TX-: U$1.84.USB3DN_TXDM5, USB6.A3, USB6.B3
- new net USB6.VBUS: D12.A, USB6.A4, USB6.A9, USB6.B4, USB6.B9
- new net VCC: D12.C, D2.C, D4.C, D5.C, D8.C, D9.C
Other:
- note added: "Keyboard: Keys: 122 Knobs: 4 KVM: Keys: 4 Knobs: 0 Media Control: Keys: 7 Knobs: 5 Total: Keys: 133 Knobs: 9 LEDs: 142 Pins: 160 + Neopixels 6*RP2040"

Commit message: Small update
Parts:
- added U6, U7: MUX.DEMUX-8X.2:2_PI3PCIE3242AZLEX, KVM-Keyboard:MUX.DEMUX-8X.2:2_PI3PCIE3242AZLEX
Changed lines of the file:
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@@
 <part name="D11" library="KVM-Keyboard" deviceset="DIODE" device="SMALL"/>
 <part name="D12" library="KVM-Keyboard" deviceset="DIODE" device="SMALL"/>
+<part name="U6" library="KVM-Keyboard" deviceset="MUX.DEMUX-8X.2:2_PI3PCIE3242AZLEX" device=""/>
+<part name="U7" library="KVM-Keyboard" deviceset="MUX.DEMUX-8X.2:2_PI3PCIE3242AZLEX" device=""/>
 </parts>
 <sheets>
@@
 <attribute name="VALUE" x="1191.26" y="169.9514" size="1.778" layer="96" rot="R180"/>
 </instance>
+<instance part="U6" gate="A" x="259.08" y="779.78" smashed="yes">
+<attribute name="NAME" x="274.32" y="806.6786" size="2.0828" layer="95" ratio="6" rot="SR0" align="center"/>
+<attribute name="VALUE" x="274.32" y="804.1386" size="2.0828" layer="96" ratio="6" rot="SR0" align="center"/>
+</instance>
+<instance part="U7" gate="A" x="848.36" y="779.78" smashed="yes">
+<attribute name="NAME" x="863.6" y="806.6786" size="2.0828" layer="95" ratio="6" rot="SR0" align="center"/>
+<attribute name="VALUE" x="863.6" y="804.1386" size="2.0828" layer="96" ratio="6" rot="SR0" align="center"/>
+</instance>
 </instances>

Commit message: Begun Neopixel testing
Connections:
- net PICO.D+: no longer U$1.42.USB2DN_DP6/PRT_DIS_P6
- net PICO.D-: no longer U$1.41.USB2DN_DM6/PRT_DIS_M6
- net USB1.R+: no longer U$1.94.USB3UP_RXDP
- net USB1.TX+: no longer U$1.91.USB3UP_TXDP
- net USB1.TX-: no longer U$1.92.USB3UP_TXDM
- net USB1RX-: no longer U$1.95.USB3UP_RXDM
- net USB2.RX+: no longer U$1.10.USB3DN_RXDP1
- net USB2.RX-: no longer U$1.11.USB3DN_RXDM1
- net USB2.TX+: no longer U$1.7.USB3DN_TXDP1
- net USB2.TX-: no longer U$1.8.USB3DN_TXDM1
- net USB3.RX+: no longer U$1.19.USB3DN_RXDP2
- net USB3.RX-: no longer U$1.20.USB3DN_RXDM2
- net USB3.TX+: no longer U$1.16.USB3DN_TXDP2
- net USB3.TX-: no longer U$1.17.USB3DN_TXDM2
- net USB4.RX+: no longer U$1.32.USB3DN_RXDP3
- net USB4.RX-: no longer U$1.33.USB3DN_RXDM3
- net USB4.TX+: no longer U$1.29.USB3DN_TXDP3
- net USB4.TX-: no longer U$1.30.USB3DN_TXDM3
- net USB5.D+: no longer U$1.34.USB2DN_DP4/PRT_DIS_P4
- net USB5.D-: no longer U$1.35.USB2DN_DM4/PRT_DIS_M4
- net USB5.RX+: no longer U$1.39.USB3DN_RXDP4
- net USB5.RX-: no longer U$1.40.USB3DN_RXDM4
- net USB5.TX+: no longer U$1.36.USB3DN_TXDP4
- net USB5.TX-: no longer U$1.37.USB3DN_TXDM4
- net USB6.D+: no longer U$1.81.USB2DN_DP5/PRT_DIS_P5
- net USB6.D-: no longer U$1.82.USB2DN_DM5/PRT_DIS_M5
- net USB6.RX+: no longer U$1.86.USB3DN_RXDP5
- net USB6.RX-: no longer U$1.87.USB3DN_RXDM5
- net USB6.TX+: no longer U$1.83.USB3DN_TXDP5
- net USB6.TX-: no longer U$1.84.USB3DN_TXDM5
